Commit message: New more inclusive launch file fixed /odom not appearing bug

File: description/gazebo_control.xacro (robot description, xacro)
@@ -6,5 +6,5 @@
             <left_joint>left_wheel_joint</left_joint>
             <right_joint>right_wheel_joint</right_joint>
-            <wheel_separation>0.2</wheel_separation>
+            <wheel_separation>0.21</wheel_separation>
             <wheel_diameter>0.104</wheel_diameter>
             <!-- Limits -->

File: description/robot.urdf.xacro (robot description, xacro)
@@ -1,5 +1,5 @@
 <?xml version="1.0"?>
-<robot xmlns:xacro="http://www.ros.org/wiki/xacro"  name="robot">
-    <xacro:include filename="robot_core.xacro" />
+<robot xmlns:xacro="http://www.ros.org/wiki/xacro"  name="tankbot_robot">
+    <xacro:include filename="robot_core_old.xacro" />
     <xacro:include filename="gazebo_control.xacro"/>
 </robot>

File: description/robot_core_old.xacro (robot description, xacro)
@@ -26,5 +26,5 @@
     <link name="chassis">
         <visual>
-            <origin xyz="0.10125 0 0.0185"/>
+            <origin xyz="0.10125 0 0.010"/>
             <geometry>
                 <mesh filename="package://tankbot/meshes/chassis.stl"/>
@@ -33,5 +33,5 @@
         </visual>
         <collision>
-            <origin xyz="0.1015 0 0.055"/>
+            <origin xyz="0.1015 0 0.05"/>
             <geometry>
                 <box size="0.215 0.201 0.10" />
@@ -49,5 +49,5 @@
         <parent link="base_link"/>
         <child link="left_wheel"/>
-        <origin xyz="0 0.105 0.0525" rpy="-${pi/2} 0 0"/>
+        <origin xyz="0 0.1105 0.044" rpy="-${pi/2} 0 0"/>
         <axis xyz="0 0 1"/>
     </joint>
@@ -60,5 +60,4 @@
         </visual>
         <collision>
-            <origin xyz="0 0.0 0.005"/>
             <geometry>
                 <cylinder radius="0.052" length="0.02"/>
@@ -75,5 +74,5 @@
         <parent link="base_link"/>
         <child link="right_wheel"/>
-        <origin xyz="0 -0.105 0.0525" rpy="${pi/2} 0 0"/>
+        <origin xyz="0 -0.10 0.044" rpy="${pi/2} 0 0"/>
         <axis xyz="0 0 -1"/>
     </joint>
@@ -86,5 +85,4 @@
         </visual>
         <collision>
-            <origin xyz="0 0.0 0.005"/>
             <geometry>
                 <cylinder radius="0.052" length="0.02"/>
@@ -101,5 +99,5 @@
         <parent link="chassis"/>
         <child link="caster_wheel"/>
-        <origin xyz="0.189 0 0.005" />
+        <origin xyz="0.189 0 -0.0025" />
     </joint>
     <link name="caster_wheel">
@@ -127,5 +125,5 @@
         <parent link="chassis"/>
         <child link="caster_wheel_back_left"/>
-        <origin xyz="0.0075 0.1337 0.0065" />
+        <origin xyz="0.0075 0.1337 -0.002" />
     </joint>
     <link name="caster_wheel_back_left">
@@ -153,5 +151,5 @@
         <parent link="chassis"/>
         <child link="caster_wheel_back_right"/>
-        <origin xyz="0.0075 -0.1337 0.0065" />
+        <origin xyz="0.0075 -0.1337 -0.002" />
     </joint>
     <link name="caster_wheel_back_right">

File: description/robot_core_simple.xacro (robot description, xacro)
@@ -26,12 +26,15 @@
     <link name="chassis">
         <visual>
-            <origin xyz="0.10125 0 0.0185"/>
+            <!-- <origin xyz="0.10125 0 0.0185"/> -->
+            <origin xyz="0.10125 0 0.055"/>
             <geometry>
-                <mesh filename="package://tankbot/meshes/chassis.stl"/>
+                <!-- <mesh filename="package://tankbot/meshes/chassis.stl"/> -->
+                <box size="0.215 0.20 0.10" />
             </geometry>
             <material name="brown"/>
         </visual>
         <collision>
-            <origin xyz="0.1015 0 0.055"/>
+            <!-- <origin xyz="0.1015 0 0.05"/> -->
+            <origin xyz="0.10125 0 0.055"/>
             <geometry>
                 <box size="0.215 0.201 0.10" />
@@ -49,5 +52,5 @@
         <parent link="base_link"/>
         <child link="left_wheel"/>
-        <origin xyz="0 0.105 0.0525" rpy="-${pi/2} 0 0"/>
+        <origin xyz="0 0.11 0.0525" rpy="-${pi/2} 0 0"/>
         <axis xyz="0 0 1"/>
     </joint>
@@ -55,10 +58,10 @@
         <visual>
             <geometry>
-                <mesh filename="package://tankbot/meshes/left_wheel_link.stl"/>
+                <!-- <mesh filename="package://tankbot/meshes/left_wheel_link.stl"/> -->
+                <cylinder radius="0.052" length="0.02"/>
             </geometry>
             <material name="white"/>
         </visual>
         <collision>
-            <origin xyz="0 0.0 0.005"/>
             <geometry>
                 <cylinder radius="0.052" length="0.02"/>
@@ -75,5 +78,5 @@
         <parent link="base_link"/>
         <child link="right_wheel"/>
-        <origin xyz="0 -0.105 0.0525" rpy="${pi/2} 0 0"/>
+        <origin xyz="0 -0.11 0.0525" rpy="${pi/2} 0 0"/>
         <axis xyz="0 0 -1"/>
     </joint>
@@ -81,10 +84,10 @@
         <visual>
             <geometry>
-                <mesh filename="package://tankbot/meshes/right_wheel_link.stl"/>
+                <!-- <mesh filename="package://tankbot/meshes/right_wheel_link.stl"/> -->
+                <cylinder radius="0.052" length="0.02"/>
             </geometry>
             <material name="white"/>
         </visual>
         <collision>
-            <origin xyz="0 0.0 0.005"/>
             <geometry>
                 <cylinder radius="0.052" length="0.02"/>
@@ -124,4 +127,5 @@
         <mu2 value="0.0001"/>
     </gazebo>
+<!--
         <joint name="caster_wheel_back_left_joint" type="fixed">
         <parent link="chassis"/>
@@ -175,4 +179,4 @@
         <mu1 value="0.0001"/>
         <mu2 value="0.0001"/>
-    </gazebo>
+    </gazebo> -->
 </robot>
