Commit message: adding gazebo launch and differential control

File: description/robot.urdf.xacro (robot description, xacro)
@@ -2,3 +2,4 @@
 <robot xmlns:xacro="http://www.ros.org/wiki/xacro"  name="robot">
     <xacro:include filename="robot_core.xacro" />
+    <xacro:include filename="gazebo_control.xacro"/>
 </robot>

File: description/robot_core.xacro (robot description, xacro)
@@ -28,5 +28,5 @@
             <origin xyz="0.10125 0 0.010"/>
             <geometry>
-                <mesh filename="package://tankbot/meshes/chassis.STL"/>
+                <mesh filename="package://tankbot/meshes/chassis.stl"/>
             </geometry>
             <material name="brown"/>
@@ -43,4 +43,7 @@
         </inertial>
     </link>
+    <gazebo reference="chassis">
+        <material>Gazebo/Blue</material>
+    </gazebo>
     <joint name="left_wheel_joint" type="continuous">
         <parent link="base_link"/>
@@ -52,5 +55,5 @@
         <visual>
             <geometry>
-                <mesh filename="package://tankbot/meshes/left_wheel_link.STL"/>
+                <mesh filename="package://tankbot/meshes/left_wheel_link.stl"/>
             </geometry>
             <material name="white"/>
@@ -65,4 +68,7 @@
         </xacro:inertial_cylinder>
     </link>
+    <gazebo reference="left_wheel">
+        <material>Gazebo/White</material>
+    </gazebo>
     <joint name="right_wheel_joint" type="continuous">
         <parent link="base_link"/>
@@ -74,5 +80,5 @@
         <visual>
             <geometry>
-                <mesh filename="package://tankbot/meshes/right_wheel_link.STL"/>
+                <mesh filename="package://tankbot/meshes/right_wheel_link.stl"/>
             </geometry>
             <material name="white"/>
@@ -87,4 +93,7 @@
         </xacro:inertial_cylinder>
     </link>
+    <gazebo reference="right_wheel">
+        <material>Gazebo/White</material>
+    </gazebo>
     <joint name="caster_wheel_joint" type="fixed">
         <parent link="chassis"/>
@@ -108,4 +117,9 @@
         </xacro:inertial_sphere>
     </link>
+    <gazebo reference="caster_wheel">
+        <material>Gazebo/Black</material>
+        <mu1 value="0.0001"/>
+        <mu2 value="0.0001"/>
+    </gazebo>
         <joint name="caster_wheel_back_left_joint" type="fixed">
         <parent link="chassis"/>
@@ -129,4 +143,9 @@
         </xacro:inertial_sphere>
     </link>
+    <gazebo reference="caster_wheel_back_left">
+        <material>Gazebo/Black</material>
+        <mu1 value="0.0001"/>
+        <mu2 value="0.0001"/>
+    </gazebo>
     <joint name="caster_wheel_back_right_joint" type="fixed">
         <parent link="chassis"/>
@@ -150,3 +169,8 @@
         </xacro:inertial_sphere>
     </link>
+   <gazebo reference="caster_wheel_back_right">
+        <material>Gazebo/Black</material>
+        <mu1 value="0.0001"/>
+        <mu2 value="0.0001"/>
+    </gazebo>
 </robot>

Commit message: Adding the lidar and camera to URDF file

File: description/robot.urdf.xacro (robot description, xacro)
@@ -1,5 +1,7 @@
 <?xml version="1.0"?>
 <robot xmlns:xacro="http://www.ros.org/wiki/xacro"  name="tankbot_robot">
-    <xacro:include filename="robot_core_old.xacro" />
+    <xacro:include filename="robot_core.xacro" />
     <xacro:include filename="gazebo_control.xacro"/>
+    <xacro:include filename="lidar.xacro"/>
+    <xacro:include filename="camera.xacro"/>
 </robot>

File: description/robot_core.xacro (robot description, xacro)
@@ -26,5 +26,5 @@
     <link name="chassis">
         <visual>
-            <origin xyz="0.10125 0 0.0185"/>
+            <origin xyz="0.10125 0 0.010"/>
             <geometry>
                 <mesh filename="package://tankbot/meshes/chassis.stl"/>
@@ -33,7 +33,11 @@
         </visual>
         <collision>
-            <origin xyz="0.1015 0 0.055"/>
+            <origin xyz="0.1015 0 0.05"/>
             <geometry>
                 <box size="0.215 0.201 0.10" />
+            </geometry>
+            <origin xyz="-0.01 0 0.01"/>
+            <geometry>
+                <box size="0.01 0.01 0.01" />
             </geometry>
         </collision>
@@ -49,5 +53,5 @@
         <parent link="base_link"/>
         <child link="left_wheel"/>
-        <origin xyz="0 0.105 0.0525" rpy="-${pi/2} 0 0"/>
+        <origin xyz="0 0.105 0.044" rpy="-${pi/2} 0 0"/>
         <axis xyz="0 0 1"/>
     </joint>
@@ -75,5 +79,5 @@
         <parent link="base_link"/>
         <child link="right_wheel"/>
-        <origin xyz="0 -0.105 0.0525" rpy="${pi/2} 0 0"/>
+        <origin xyz="0 -0.105 0.044" rpy="${pi/2} 0 0"/>
         <axis xyz="0 0 -1"/>
     </joint>
@@ -101,5 +105,5 @@
         <parent link="chassis"/>
         <child link="caster_wheel"/>
-        <origin xyz="0.189 0 0.005" />
+        <origin xyz="0.189 0 -0.0025" />
     </joint>
     <link name="caster_wheel">
@@ -127,5 +131,5 @@
         <parent link="chassis"/>
         <child link="caster_wheel_back_left"/>
-        <origin xyz="0.0075 0.1337 0.0065" />
+        <origin xyz="0.0075 0.1337 -0.002" />
     </joint>
     <link name="caster_wheel_back_left">
@@ -153,5 +157,5 @@
         <parent link="chassis"/>
         <child link="caster_wheel_back_right"/>
-        <origin xyz="0.0075 -0.1337 0.0065" />
+        <origin xyz="0.0075 -0.1337 -0.002" />
     </joint>
     <link name="caster_wheel_back_right">

Commit message: Fixing visuals and meshes for gazebo simulation

File: description/robot.urdf.xacro (robot description, xacro)
@@ -1,4 +1,4 @@
 <?xml version="1.0"?>
-<robot xmlns:xacro="http://www.ros.org/wiki/xacro"  name="tankbot_robot">
+<robot xmlns:xacro="http://www.ros.org/wiki/xacro"  name="tankbot">
     <xacro:include filename="robot_core.xacro" />
     <xacro:include filename="gazebo_control.xacro"/>

File: description/tankbot.urdf (robot description, URDF)
Before this commit: robot tankbot_robot, 7 links, 6 joints
Links:
- added link camera_frame, mass 0.04; collision box size=0.035 0.035 0.035; visual mesh filename=package://tankbot/meshes/camera.STL
- added link laser_frame, mass 0.08; collision cylinder length=0.055 radius=0.035; visual mesh filename=package://tankbot/meshes/lidar.STL
Joints:
- added joint camera_joint: type fixed, parent chassis, child camera_frame, origin xyz=0.195 0 0.095 rpy=0 0 0
- added joint laser_joint: type fixed, parent chassis, child laser_frame, origin xyz=0.035 0 0.135 rpy=0 0 0
- joint left_wheel_joint: origin xyz=0 0.1105 0.044 rpy=-1.5707963267948966 0 0 -> xyz=0 0.105 0.044 rpy=-1.5707963267948966 0 0
- joint right_wheel_joint: origin xyz=0 -0.10 0.044 rpy=1.5707963267948966 0 0 -> xyz=0 -0.105 0.044 rpy=1.5707963267948966 0 0
