Commit message: Updating URDF vidual and inertial measurements

File: description/camera.xacro (robot description, xacro)
@@ -8,18 +8,19 @@
     <link name="camera_frame">
         <visual>
+            <origin xyz="-0.094 0 -0.085"/>
             <geometry>
-                <box size="0.02 0.02 0.02"/>
+                <mesh filename="package://tankbot/meshes/camera.STL"/>
             </geometry>
             <material name="blue"/>
         </visual>
         <collision>
+            <origin xyz="0.195 0 0.095" rpy="0 0 0"/> -->
             <geometry>
-                <box size="0.02 0.02 0.02" />
+                <box size="0.035 0.035 0.035" />
             </geometry>
         </collision>
-        <inertial>
-            <mass value="1"/>
-            <inertia ixx="0.00556875" ixy="0.0" ixz="0.00489336" iyy="0.025445" iyz="0.0" izz="0.0276345"/>
-        </inertial>
+        <xacro:inertial_box mass="0.04" x="0.035" y="0.035" z="0.035">
+            <origin xyz="0 0 0" rpy="0 0 0"/>
+        </xacro:inertial_box>
     </link>
 </robot>

File: description/lidar.xacro (robot description, xacro)
@@ -4,11 +4,11 @@
         <parent link="chassis"/>
         <child link="laser_frame"/>
-        <origin xyz="0.005 0 0.13" rpy="0 0 0"/>
+        <origin xyz="0.035 0 0.135" rpy="0 0 0"/>
     </joint>
     <link name="laser_frame">
         <visual>
-            <origin xyz="0.035 0 0.0225"/>
+            <origin xyz="0.066 0 -0.125"/>
             <geometry>
-                <cylinder radius ="0.035" length="0.055" />
+                <mesh filename="package://tankbot/meshes/lidar.STL"/>
             </geometry>
             <material name="black"/>
@@ -20,8 +20,7 @@
             </geometry>
         </collision>
-        <inertial>
-            <mass value="1"/>
-            <inertia ixx="0.00556875" ixy="0.0" ixz="0.00489336" iyy="0.025445" iyz="0.0" izz="0.0276345"/>
-        </inertial>
+        <xacro:inertial_cylinder mass="0.08" length="0.02" radius="0.052">
+            <origin xyz="0 0 0" rpy="0 0 0"/>
+        </xacro:inertial_cylinder>
     </link>
 </robot>

Commit message: Adding lidar and camera functionality to gazebo

File: description/camera.xacro (robot description, xacro)
@@ -15,12 +15,41 @@
         </visual>
         <collision>
-            <origin xyz="0.195 0 0.095" rpy="0 0 0"/> -->
+            <origin xyz="-0.005 0 0" rpy="0 0 0"/>
             <geometry>
                 <box size="0.035 0.035 0.035" />
             </geometry>
         </collision>
-        <xacro:inertial_box mass="0.04" x="0.035" y="0.035" z="0.035">
+        <xacro:inertial_box mass="0.02" x="0.035" y="0.035" z="0.035">
             <origin xyz="0 0 0" rpy="0 0 0"/>
         </xacro:inertial_box>
     </link>
+    <joint name="camera_optical_joint" type="fixed">
+        <parent link="camera_frame"/>
+        <child link="camera_optical_link"/>
+        <origin xyz="0 0 0.0125" rpy="${-pi/2} 0 ${-pi/2}"/>
+    </joint>
+    <link name="camera_optical_link"></link>
+    <gazebo reference="camera_frame">
+        <material>Gazebo/White</material>
+        <sensor name="camera" type="camera">
+            <pose> 0 0 0 0 0 0 </pose>
+            <visualize>true</visualize>
+            <update_rate>10</update_rate>
+            <camera>
+                <horizontal_fov>1.089</horizontal_fov>
+                <image>
+                    <format>R8G8B8</format>
+                    <width>640</width>
+                    <height>480</height>
+                </image>
+                <clip>
+                    <near>0.05</near>
+                    <far>8.0</far>
+                </clip>
+            </camera>
+            <plugin name="camera_controller" filename="libgazebo_ros_camera.so">
+                <frame_name>camera_optical_link</frame_name>
+            </plugin>
+        </sensor>
+    </gazebo>
 </robot>

File: description/lidar.xacro (robot description, xacro)
@@ -4,9 +4,9 @@
         <parent link="chassis"/>
         <child link="laser_frame"/>
-        <origin xyz="0.035 0 0.135" rpy="0 0 0"/>
+        <origin xyz="0.035 0 0.165" rpy="0 0 0"/>
     </joint>
     <link name="laser_frame">
         <visual>
-            <origin xyz="0.066 0 -0.125"/>
+            <origin xyz="0.066 0 -0.155"/>
             <geometry>
                 <mesh filename="package://tankbot/meshes/lidar.STL"/>
@@ -15,5 +15,5 @@
         </visual>
         <collision>
-            <origin xyz="0.035 0 0.0225"/>
+            <origin xyz="0 0 -0.03"/>
             <geometry>
                 <cylinder radius ="0.035" length="0.055" />
@@ -24,3 +24,31 @@
         </xacro:inertial_cylinder>
     </link>
+    <gazebo reference="laser_frame">
+        <material>Gazebo/Black</material>
+        <sensor name="laser" type="ray">
+            <pose> 0 0 0 0 0 0 </pose>
+            <visualize>true</visualize>
+            <update_rate>10</update_rate>
+            <ray>
+                <scan>
+                    <horizontal>
+                        <samples>360</samples>
+                        <min_angle>-3.14</min_angle>
+                        <max_angle>3.14</max_angle>
+                    </horizontal>
+                </scan>
+                <range>
+                    <min>0.3</min>
+                    <max>12</max>
+                </range>
+            </ray>
+            <plugin name="laser_controller" filename="libgazebo_ros_ray_sensor.so">
+                <ros>
+                    <argument>~/out:=scan</argument>
+                </ros>
+                <output_type>sensor_msgs/LaserScan</output_type>
+                <frame_name>laser_frame</frame_name>
+            </plugin>
+        </sensor>
+    </gazebo>
 </robot>

File: description/tankbot.urdf (robot description, URDF)
Before this commit: robot tankbot, 9 links, 8 joints
Links:
- added link camera_optical_link
- link camera_frame: mass 0.04 -> 0.02
Joints:
- added joint camera_optical_joint: type fixed, parent camera_frame, child camera_optical_link, origin xyz=0 0 0.0125 rpy=-1.5707963267948966 0 -1.5707963267948966
- joint laser_joint: origin xyz=0.035 0 0.135 rpy=0 0 0 -> xyz=0.035 0 0.165 rpy=0 0 0
