Commit message: Updating URDF visuals

File: description/robot_core.xacro (robot description, xacro)
@@ -26,14 +26,14 @@
     <link name="chassis">
         <visual>
-            <origin xyz="0.105 0 0.050"/>
+            <origin xyz="0.10125 0 0.010"/>
             <geometry>
-                <box size="0.21 0.201 0.10" />
+                <mesh filename="package://tankbot/meshes/chassis.STL"/>
             </geometry>
             <material name="brown"/>
         </visual>
         <collision>
-            <origin xyz="0.105 0 0.050"/>
+            <origin xyz="0.1015 0 0.05"/>
             <geometry>
-                <box size="0.21 0.201 0.10" />
+                <box size="0.215 0.201 0.10" />
             </geometry>
         </collision>
@@ -51,5 +51,5 @@
         <visual>
             <geometry>
-                <cylinder radius="0.052" length="0.02"/>
+                <mesh filename="package://tankbot/meshes/left_wheel_link.STL"/>
             </geometry>
             <material name="white"/>
@@ -67,5 +67,5 @@
         <parent link="base_link"/>
         <child link="right_wheel"/>
-        <origin xyz="0 -0.1105 0.044" rpy="${pi/2} 0 0"/>
+        <origin xyz="0 -0.10 0.044" rpy="${pi/2} 0 0"/>
         <axis xyz="0 0 -1"/>
     </joint>
@@ -73,5 +73,5 @@
         <visual>
             <geometry>
-                <cylinder radius="0.052" length="0.02"/>
+                <mesh filename="package://tankbot/meshes/right_wheel_link.STL"/>
             </geometry>
             <material name="white"/>
@@ -89,10 +89,10 @@
         <parent link="chassis"/>
         <child link="caster_wheel"/>
-        <origin xyz="0.202 0 0" />
+        <origin xyz="0.189 0 -0.0025" />
     </joint>
     <link name="caster_wheel">
         <visual>
             <geometry>
-                <sphere radius="0.008"/>
+                <sphere radius="0.005"/>
             </geometry>
             <material name="black"/>
@@ -100,5 +100,5 @@
         <collision>
             <geometry>
-                <sphere radius="0.008"/>
+                <sphere radius="0.005"/>
             </geometry>
         </collision>

Commit message: Updating URDF intertial Values and back caster wheels

File: description/robot_core.xacro (robot description, xacro)
@@ -38,7 +38,8 @@
             </geometry>
         </collision>
-        <xacro:inertial_box mass="0.5" x="0.21" y="0.201" z="0.1">
-            <origin xyz="0.105 0 0.050" rpy="0 0 0"/>
-        </xacro:inertial_box>
+        <inertial>
+            <mass value="1"/>
+            <inertia ixx="0.00556875" ixy="0.0" ixz="0.00489336" iyy="0.025445" iyz="0.0" izz="0.0276345"/>
+        </inertial>
     </link>
     <joint name="left_wheel_joint" type="continuous">
@@ -60,5 +61,5 @@
             </geometry>
         </collision>
-        <xacro:inertial_cylinder mass="0.1" length="0.02" radius="0.052">
+        <xacro:inertial_cylinder mass="0.08" length="0.02" radius="0.052">
             <origin xyz="0 0 0" rpy="0 0 0"/>
         </xacro:inertial_cylinder>
@@ -82,5 +83,5 @@
             </geometry>
         </collision>
-        <xacro:inertial_cylinder mass="0.1" length="0.02" radius="0.052">
+        <xacro:inertial_cylinder mass="0.08" length="0.02" radius="0.052">
             <origin xyz="0 0 0" rpy="0 0 0"/>
         </xacro:inertial_cylinder>
@@ -103,5 +104,47 @@
             </geometry>
         </collision>
-        <xacro:inertial_sphere mass="0.01" radius="0.008">
+        <xacro:inertial_sphere mass="0.004" radius="0.005">
+            <origin xyz="0 0 0" rpy="0 0 0"/>
+        </xacro:inertial_sphere>
+    </link>
+        <joint name="caster_wheel_back_left_joint" type="fixed">
+        <parent link="chassis"/>
+        <child link="caster_wheel_back_left"/>
+        <origin xyz="0.0075 0.1337 -0.002" />
+    </joint>
+    <link name="caster_wheel_back_left">
+        <visual>
+            <geometry>
+                <sphere radius="0.0065"/>
+            </geometry>
+            <material name="black"/>
+        </visual>
+        <collision>
+            <geometry>
+                <sphere radius="0.0065"/>
+            </geometry>
+        </collision>
+        <xacro:inertial_sphere mass="0.005" radius="0.0065">
+            <origin xyz="0 0 0" rpy="0 0 0"/>
+        </xacro:inertial_sphere>
+    </link>
+    <joint name="caster_wheel_back_right_joint" type="fixed">
+        <parent link="chassis"/>
+        <child link="caster_wheel_back_right"/>
+        <origin xyz="0.0075 -0.1337 -0.002" />
+    </joint>
+    <link name="caster_wheel_back_right">
+        <visual>
+            <geometry>
+                <sphere radius="0.0065"/>
+            </geometry>
+            <material name="black"/>
+        </visual>
+        <collision>
+            <geometry>
+                <sphere radius="0.0065"/>
+            </geometry>
+        </collision>
+        <xacro:inertial_sphere mass="0.005" radius="0.0065">
             <origin xyz="0 0 0" rpy="0 0 0"/>
         </xacro:inertial_sphere>

Commit message: updating xacro files

File: description/robot_core.xacro (robot description, xacro)
@@ -26,5 +26,5 @@
     <link name="chassis">
         <visual>
-            <origin xyz="0.10125 0 0.010"/>
+            <origin xyz="0.10125 0 0.0185"/>
             <geometry>
                 <mesh filename="package://tankbot/meshes/chassis.stl"/>
@@ -49,5 +49,5 @@
         <parent link="base_link"/>
         <child link="left_wheel"/>
-        <origin xyz="0 0.1105 0.044" rpy="-${pi/2} 0 0"/>
+        <origin xyz="0 0.105 0.0525" rpy="-${pi/2} 0 0"/>
         <axis xyz="0 0 1"/>
     </joint>
@@ -74,5 +74,5 @@
         <parent link="base_link"/>
         <child link="right_wheel"/>
-        <origin xyz="0 -0.10 0.044" rpy="${pi/2} 0 0"/>
+        <origin xyz="0 -0.105 0.0525" rpy="${pi/2} 0 0"/>
         <axis xyz="0 0 -1"/>
     </joint>
@@ -99,5 +99,5 @@
         <parent link="chassis"/>
         <child link="caster_wheel"/>
-        <origin xyz="0.189 0 -0.0025" />
+        <origin xyz="0.189 0 0.005" />
     </joint>
     <link name="caster_wheel">
@@ -125,5 +125,5 @@
         <parent link="chassis"/>
         <child link="caster_wheel_back_left"/>
-        <origin xyz="0.0075 0.1337 -0.002" />
+        <origin xyz="0.0075 0.1337 0.0065" />
     </joint>
     <link name="caster_wheel_back_left">
@@ -151,5 +151,5 @@
         <parent link="chassis"/>
         <child link="caster_wheel_back_right"/>
-        <origin xyz="0.0075 -0.1337 -0.002" />
+        <origin xyz="0.0075 -0.1337 0.0065" />
     </joint>
     <link name="caster_wheel_back_right">

Commit message: Stateted SLAM in gazebo and fixed some issues

File: description/robot_core.xacro (robot description, xacro)
@@ -18,4 +18,11 @@
     </material>
     <link name="base_link">
+    </link>
+    <joint name="base_footprint_joint" type="fixed">
+        <parent link="base_link"/>
+        <child link="base_footprint"/>
+        <origin xyz="0 0 0" rpy="0 0 0"/>
+    </joint>
+    <link name="base_footprint">
     </link>
     <joint name="chassis_joint" type="fixed">

File: description/tankbot.urdf (robot description, URDF)
Before this commit: robot tankbot, 10 links, 9 joints
Links:
- added link base_footprint
Joints:
- added joint base_footprint_joint: type fixed, parent base_link, child base_footprint, origin xyz=0 0 0 rpy=0 0 0
